Commit message: Message de commit des modifications dans robot.urdf.xacro

File: description/robot.urdf.xacro (robot description, xacro)
@@ -44,3 +44,37 @@
     <origin xyz="-0.1 0 0"/>
   </joint>
+   <!-- Définition du joint entre chassis et le bras gauche -->
+  <joint    name="left_wheel_joint" type="continuous">
+    <parent link="base_link"/>
+    <child  link="left_wheel"/>
+    <origin  xyz="0 0.175 0" rpy="-${pi/2} 0 0"/>
+    <axis    xyz="0 0 1"/>
+  </joint>
+<!-- Définition du lien bras gauche du chassis -->
+  <link name="left_wheel">
+    <visual>
+      <origin xyz="0.15 0 0.75"/>
+      <geometry>
+        <cylinder radius="0.05" length="0.04"/>
+      </geometry>
+      <material name="blue"/>
+    </visual>
+  </link>
+   <!-- Définition du joint entre chassis et le bras droit -->
+  <joint    name="left_wheel_joint" type="continuous">
+    <parent link="base_link"/>
+    <child  link="right_wheel"/>
+    <origin  xyz="0 -0.175 0" rpy="${pi/2} 0 0"/>
+    <axis    xyz="0 0 -1"/>
+  </joint>
+<!-- Définition du lien bras droit du chassis -->
+  <link name="right_wheel">
+    <visual>
+      <origin xyz="0.15 0 0.75"/>
+      <geometry>
+        <cylinder radius="0.05" length="0.04"/>
+      </geometry>
+      <material name="blue"/>
+    </visual>
+  </link>
 </robot>

Commit message: Message de commit des modifications dans robot.urdf.xacro

File: description/robot.urdf.xacro (robot description, xacro)
@@ -62,5 +62,5 @@
   </link>
    <!-- Définition du joint entre chassis et le bras droit -->
-  <joint    name="left_wheel_joint" type="continuous">
+  <joint    name="right_wheel_joint" type="continuous">
     <parent link="base_link"/>
     <child  link="right_wheel"/>

Commit message: Modifications des fichiers URDF et Xacro

File: description/robot.urdf.xacro (robot description, xacro)
@@ -31,5 +31,5 @@
   <link name="chassis">
     <visual>
-      <origin xyz="0.15 0 0.75"/>
+      <origin xyz="0 0 0"/>
       <geometry>
         <box size="0.3 0.3 0.15"/>
@@ -42,17 +42,17 @@
     <parent link="base_link"/>
     <child link="chassis"/>
-    <origin xyz="-0.1 0 0"/>
+    <origin xyz="0 0 0"/>
   </joint>
-   <!-- Définition du joint entre chassis et le bras gauche -->
-  <joint    name="left_wheel_joint" type="continuous">
-    <parent link="base_link"/>
-    <child  link="left_wheel"/>
-    <origin  xyz="0 0.175 0" rpy="-${pi/2} 0 0"/>
-    <axis    xyz="0 0 1"/>
+  <!-- Définition du joint entre chassis et le bras gauche -->
+  <joint name="left_wheel_joint" type="continuous">
+    <parent link="chassis"/>
+    <child link="left_wheel"/>
+    <origin xyz="0 0.15 0" rpy="0 0 ${pi/2}"/>
+    <axis xyz="0 1 0"/>
   </joint>
-<!-- Définition du lien bras gauche du chassis -->
+  <!-- Définition du lien bras gauche du chassis -->
   <link name="left_wheel">
     <visual>
-      <origin xyz="0.15 0 0.75"/>
+      <origin xyz="0 0 0"/>
       <geometry>
         <cylinder radius="0.05" length="0.04"/>
@@ -61,15 +61,15 @@
     </visual>
   </link>
-   <!-- Définition du joint entre chassis et le bras droit -->
-  <joint    name="right_wheel_joint" type="continuous">
-    <parent link="base_link"/>
-    <child  link="right_wheel"/>
-    <origin  xyz="0 -0.175 0" rpy="${pi/2} 0 0"/>
-    <axis    xyz="0 0 -1"/>
+  <!-- Définition du joint entre chassis et le bras droit -->
+  <joint name="right_wheel_joint" type="continuous">
+    <parent link="chassis"/>
+    <child link="right_wheel"/>
+    <origin xyz="0 -0.15 0" rpy="0 0 ${pi/2}"/>
+    <axis xyz="0 1 0"/>
   </joint>
-<!-- Définition du lien bras droit du chassis -->
+  <!-- Définition du lien bras droit du chassis -->
   <link name="right_wheel">
     <visual>
-      <origin xyz="0.15 0 0.75"/>
+      <origin xyz="0 0 0"/>
       <geometry>
         <cylinder radius="0.05" length="0.04"/>

Commit message: Description succincte de vos modifications_1.1

File: description/robot.urdf.xacro (robot description, xacro)
@@ -1,4 +1,6 @@
 <?xml version="1.0"?>
 <robot xmlns:xacro="http://www.ros.org/wiki/xacro" name="robot">
+  <!-- Inclusion de xacro pour utiliser les macros et les constantes -->
+  <xacro:property name="pi" value="3.141592653589793"/>
   <!-- Définition des matériaux -->
   <material name="white">
@@ -48,6 +50,6 @@
     <parent link="chassis"/>
     <child link="left_wheel"/>
-    <origin xyz="0 0.15 0" rpy="0 0 ${pi/2}"/>
-    <axis xyz="0 1 0"/>
+    <origin xyz="0 0.175 0" rpy="-${pi/2} 0 0"/>
+    <axis xyz="0 0 1"/>
   </joint>
   <!-- Définition du lien bras gauche du chassis -->
@@ -65,6 +67,6 @@
     <parent link="chassis"/>
     <child link="right_wheel"/>
-    <origin xyz="0 -0.15 0" rpy="0 0 ${pi/2}"/>
-    <axis xyz="0 1 0"/>
+    <origin xyz="0 -0.175 0" rpy="${pi/2} 0 0"/>
+    <axis xyz="0 0 -1"/>
   </joint>
   <!-- Définition du lien bras droit du chassis -->

Commit message: Description succincte de vos modifications_1.2

File: description/robot.urdf.xacro (robot description, xacro)
@@ -1,7 +1,5 @@
 <?xml version="1.0"?>
 <robot xmlns:xacro="http://www.ros.org/wiki/xacro" name="robot">
-  <!-- Inclusion de xacro pour utiliser les macros et les constantes -->
-  <xacro:property name="pi" value="3.141592653589793"/>
-  <!-- Définition des matériaux -->
+    <!-- Définition des matériaux -->
   <material name="white">
     <color rgba="1 1 1 1"/>

Commit message: Description succincte de vos modifications_origin_chassis

File: description/robot.urdf.xacro (robot description, xacro)
@@ -31,5 +31,5 @@
   <link name="chassis">
     <visual>
-      <origin xyz="0 0 0"/>
+      <origin xyz="0.15 0 0.75"/>
       <geometry>
         <box size="0.3 0.3 0.15"/>

Commit message: Description succincte de vos modifications_origin_chassis2

File: description/robot.urdf.xacro (robot description, xacro)
@@ -31,5 +31,5 @@
   <link name="chassis">
     <visual>
-      <origin xyz="0.15 0 0.75"/>
+      <origin xyz="0.15 0 0.075"/>
       <geometry>
         <box size="0.3 0.3 0.15"/>
@@ -42,5 +42,5 @@
     <parent link="base_link"/>
     <child link="chassis"/>
-    <origin xyz="0 0 0"/>
+    <origin xyz="-0.1 0 0"/>
   </joint>
   <!-- Définition du joint entre chassis et le bras gauche -->

File: description/robot_core.xacro (robot description, xacro)
@@ -1,5 +1,5 @@
 <?xml version="1.0"?>
 <robot xmlns:xacro="http://www.ros.org/wiki/xacro" name="robot">
-  <!-- Définition des matériaux -->
+    <!-- Définition des matériaux -->
   <material name="white">
     <color rgba="1 1 1 1"/>
@@ -14,18 +14,22 @@
     <color rgba="0 0 0 1"/>
   </material>
+  <!-- Définition du lien world -->
+  <link name="world">
+    <!-- Contenu du lien world -->
+  </link>
   <!-- Définition du lien de base -->
   <link name="base_link">
     <!-- Contenu du lien base_link -->
   </link>
-  <!-- Définition du joint base_link -->
+  <!-- Définition du joint base_joint -->
   <joint name="base_joint" type="fixed">
     <parent link="world"/>
     <child link="base_link"/>
-    <origin xyz="0 0 0" rpy="0 0 0"/>
+    <origin rpy="0 0 0" xyz="0 0 0"/>
   </joint>
   <!-- Définition du lien chassis -->
   <link name="chassis">
     <visual>
-      <origin xyz="0.15 0 0.75"/>
+      <origin xyz="0.15 0 0.075"/>
       <geometry>
         <box size="0.3 0.3 0.15"/>
@@ -40,3 +44,37 @@
     <origin xyz="-0.1 0 0"/>
   </joint>
+  <!-- Définition du joint entre chassis et le bras gauche -->
+  <joint name="left_wheel_joint" type="continuous">
+    <parent link="chassis"/>
+    <child link="left_wheel"/>
+    <origin xyz="0 0.175 0" rpy="-${pi/2} 0 0"/>
+    <axis xyz="0 0 1"/>
+  </joint>
+  <!-- Définition du lien bras gauche du chassis -->
+  <link name="left_wheel">
+    <visual>
+      <origin xyz="0 0 0"/>
+      <geometry>
+        <cylinder radius="0.05" length="0.04"/>
+      </geometry>
+      <material name="blue"/>
+    </visual>
+  </link>
+  <!-- Définition du joint entre chassis et le bras droit -->
+  <joint name="right_wheel_joint" type="continuous">
+    <parent link="chassis"/>
+    <child link="right_wheel"/>
+    <origin xyz="0 -0.175 0" rpy="${pi/2} 0 0"/>
+    <axis xyz="0 0 -1"/>
+  </joint>
+  <!-- Définition du lien bras droit du chassis -->
+  <link name="right_wheel">
+    <visual>
+      <origin xyz="0 0 0"/>
+      <geometry>
+        <cylinder radius="0.05" length="0.04"/>
+      </geometry>
+      <material name="blue"/>
+    </visual>
+  </link>
 </robot>

Commit message: origine_des_roues_base_link

File: description/robot.urdf.xacro (robot description, xacro)
@@ -46,5 +46,5 @@
   <!-- Définition du joint entre chassis et le bras gauche -->
   <joint name="left_wheel_joint" type="continuous">
-    <parent link="chassis"/>
+    <parent link="base_link"/>
     <child link="left_wheel"/>
     <origin xyz="0 0.175 0" rpy="-${pi/2} 0 0"/>
@@ -63,5 +63,5 @@
   <!-- Définition du joint entre chassis et le bras droit -->
   <joint name="right_wheel_joint" type="continuous">
-    <parent link="chassis"/>
+    <parent link="base_link"/>
     <child link="right_wheel"/>
     <origin xyz="0 -0.175 0" rpy="${pi/2} 0 0"/>

File: description/robot_core.xacro (robot description, xacro)
@@ -46,5 +46,5 @@
   <!-- Définition du joint entre chassis et le bras gauche -->
   <joint name="left_wheel_joint" type="continuous">
-    <parent link="chassis"/>
+    <parent link="base_link"/>
     <child link="left_wheel"/>
     <origin xyz="0 0.175 0" rpy="-${pi/2} 0 0"/>
@@ -63,5 +63,5 @@
   <!-- Définition du joint entre chassis et le bras droit -->
   <joint name="right_wheel_joint" type="continuous">
-    <parent link="chassis"/>
+    <parent link="base_link"/>
     <child link="right_wheel"/>
     <origin xyz="0 -0.175 0" rpy="${pi/2} 0 0"/>

Commit message: collision

File: description/robot.urdf.xacro (robot description, xacro)
@@ -78,3 +78,18 @@
     </visual>
   </link>
+<!-- Définition du joint entre chassis et la roulette(caster_wheel) -->
+  <joint name="caster_wheel_joint" type="continuous">
+    <parent link="chassis"/>
+    <child link="caster_wheel"/>
+    <origin xyz="0.24 0 0" rpy="${pi/2} 0 0"/>
+  </joint>
+  <!-- Définition du lien la roulette(caster_wheel) -->
+  <link name="caster_wheel">
+    <visual>
+      <geometry>
+        <sphere radius="0.05" />
+      </geometry>
+      <material name="black"/>
+    </visual>
+  </link>
 </robot>

File: description/robot_core.xacro (robot description, xacro)
@@ -1,4 +1,5 @@
 <?xml version="1.0"?>
 <robot xmlns:xacro="http://www.ros.org/wiki/xacro" name="robot">
+  <xacro:include filename="inertial_macros.xacro"/>
     <!-- Définition des matériaux -->
   <material name="white">
@@ -37,4 +38,13 @@
       <material name="white"/>
     </visual>
+    <collision>
+      <origin xyz="0.15 0 0.075"/>
+      <geometry>
+        <box size="0.3 0.3 0.15"/>
+      </geometry>
+    </collision>
+    <xacro:inertial_box mass="0.5" x="0.3" y="0.3" z="0.15">
+      <origin xyz="0.15 0 0.075" rpy="0 0 0"/>
+      </xacro:inertial_box>
   </link>
   <!-- Définition du joint entre base_link et chassis -->
@@ -60,4 +70,13 @@
       <material name="blue"/>
     </visual>
+    <collision>
+      <origin xyz="0 0 0"/>
+      <geometry>
+        <cylinder radius="0.05" length="0.04"/>
+      </geometry>
+    </collision>
+    <xacro:inertial_cylinder mass="0.1" length="0.04" radius="0.05">
+      <origin xyz="0 0 0" rpy="0 0 0"/>
+    </xacro:inertial_cylinder>
   </link>
   <!-- Définition du joint entre chassis et le bras droit -->
@@ -77,4 +96,36 @@
       <material name="blue"/>
     </visual>
+    <collision>
+      <origin xyz="0 0 0"/>
+      <geometry>
+        <cylinder radius="0.05" length="0.04"/>
+      </geometry>
+    </collision>
+    <xacro:inertial_cylinder mass="0.1" length="0.04" radius="0.05">
+      <origin xyz="0 0 0" rpy="0 0 0"/>
+    </xacro:inertial_cylinder>
+  </link>
+<!-- Définition du joint entre chassis et la roulette(caster_wheel) -->
+  <joint name="caster_wheel_joint" type="continuous">
+    <parent link="chassis"/>
+    <child link="caster_wheel"/>
+    <origin xyz="0.24 0 0" rpy="${pi/2} 0 0"/>
+  </joint>
+  <!-- Définition du lien la roulette(caster_wheel) -->
+  <link name="caster_wheel">
+    <visual>
+      <geometry>
+        <sphere radius="0.05" />
+      </geometry>
+      <material name="black"/>
+    </visual>
+    <collision>
+      <geometry>
+        <sphere radius="0.05" />
+      </geometry>
+    </collision>
+    <xacro:inertial_sphere mass="0.1"  radius="0.05">
+      <origin xyz="0 0 0" rpy="0 0 0"/>
+    </xacro:inertial_sphere>
   </link>
 </robot>
