Commit message: Description succincte de vos modifications

File: description/robot.urdf (robot description, URDF)
Before this commit: robot robot, 1 links, 0 joints
Links:
- added link chassis; visual box size=0.3 0.3 0.15
Joints:
- added joint base_joint: type fixed, parent world, child base_link, origin xyz=0 0 0 rpy=0 0 0
- added joint chassis_joint: type fixed, parent base_link, child chassis, origin xyz=-0.1 0 0

File: description/robot.urdf.xacro (robot description, xacro)
@@ -1,4 +1,46 @@
 <?xml version="1.0"?>
-<robot xmlns:xacro="http://www.ros.org/wiki/xacro"  name="robot">
-    <xacro:include filename="robot_core.xacro" />
+<robot xmlns:xacro="http://www.ros.org/wiki/xacro" name="robot">
+  <!-- Définition des matériaux -->
+  <material name="white">
+    <color rgba="1 1 1 1"/>
+  </material>
+  <material name="orange">
+    <color rgba="1 0.3 0.1 1"/>
+  </material>
+  <material name="blue">
+    <color rgba="0.2 0.2 1 1"/>
+  </material>
+  <material name="black">
+    <color rgba="0 0 0 1"/>
+  </material>
+  <!-- Définition du lien world -->
+  <link name="world">
+    <!-- Contenu du lien world -->
+  </link>
+  <!-- Définition du lien de base -->
+  <link name="base_link">
+    <!-- Contenu du lien base_link -->
+  </link>
+  <!-- Définition du joint base_joint -->
+  <joint name="base_joint" type="fixed">
+    <parent link="world"/>
+    <child link="base_link"/>
+    <origin rpy="0 0 0" xyz="0 0 0"/>
+  </joint>
+  <!-- Définition du lien chassis -->
+  <link name="chassis">
+    <visual>
+      <origin xyz="0.15 0 0.75"/>
+      <geometry>
+        <box size="0.3 0.3 0.15"/>
+      </geometry>
+      <material name="white"/>
+    </visual>
+  </link>
+  <!-- Définition du joint entre base_link et chassis -->
+  <joint name="chassis_joint" type="fixed">
+    <parent link="base_link"/>
+    <child link="chassis"/>
+    <origin xyz="-0.1 0 0"/>
+  </joint>
 </robot>

Commit message: derniere_mise_a_jour_robot.urdf.xacro

File: description/robot.urdf (robot description, URDF)
Before this commit: robot robot, 6 links, 5 joints
Links:
- link caster_wheel: geometry collision sphere radius=0.05; visual sphere radius=0.05
- link chassis: geometry collision box size=0.3 0.3 0.15; visual box size=0.3 0.3 0.15
- link left_wheel: geometry collision cylinder length=0.04 radius=0.05; visual cylinder length=0.04 radius=0.05
- link right_wheel: geometry collision cylinder length=0.04 radius=0.05; visual cylinder length=0.04 radius=0.05

File: description/robot.urdf.xacro (robot description, xacro)
@@ -1,95 +1,4 @@
 <?xml version="1.0"?>
 <robot xmlns:xacro="http://www.ros.org/wiki/xacro" name="robot">
-    <!-- Définition des matériaux -->
-  <material name="white">
-    <color rgba="1 1 1 1"/>
-  </material>
-  <material name="orange">
-    <color rgba="1 0.3 0.1 1"/>
-  </material>
-  <material name="blue">
-    <color rgba="0.2 0.2 1 1"/>
-  </material>
-  <material name="black">
-    <color rgba="0 0 0 1"/>
-  </material>
-  <!-- Définition du lien world -->
-  <link name="world">
-    <!-- Contenu du lien world -->
-  </link>
-  <!-- Définition du lien de base -->
-  <link name="base_link">
-    <!-- Contenu du lien base_link -->
-  </link>
-  <!-- Définition du joint base_joint -->
-  <joint name="base_joint" type="fixed">
-    <parent link="world"/>
-    <child link="base_link"/>
-    <origin rpy="0 0 0" xyz="0 0 0"/>
-  </joint>
-  <!-- Définition du lien chassis -->
-  <link name="chassis">
-    <visual>
-      <origin xyz="0.15 0 0.075"/>
-      <geometry>
-        <box size="0.3 0.3 0.15"/>
-      </geometry>
-      <material name="white"/>
-    </visual>
-  </link>
-  <!-- Définition du joint entre base_link et chassis -->
-  <joint name="chassis_joint" type="fixed">
-    <parent link="base_link"/>
-    <child link="chassis"/>
-    <origin xyz="-0.1 0 0"/>
-  </joint>
-  <!-- Définition du joint entre chassis et le bras gauche -->
-  <joint name="left_wheel_joint" type="continuous">
-    <parent link="base_link"/>
-    <child link="left_wheel"/>
-    <origin xyz="0 0.175 0" rpy="-${pi/2} 0 0"/>
-    <axis xyz="0 0 1"/>
-  </joint>
-  <!-- Définition du lien bras gauche du chassis -->
-  <link name="left_wheel">
-    <visual>
-      <origin xyz="0 0 0"/>
-      <geometry>
-        <cylinder radius="0.05" length="0.04"/>
-      </geometry>
-      <material name="blue"/>
-    </visual>
-  </link>
-  <!-- Définition du joint entre chassis et le bras droit -->
-  <joint name="right_wheel_joint" type="continuous">
-    <parent link="base_link"/>
-    <child link="right_wheel"/>
-    <origin xyz="0 -0.175 0" rpy="${pi/2} 0 0"/>
-    <axis xyz="0 0 -1"/>
-  </joint>
-  <!-- Définition du lien bras droit du chassis -->
-  <link name="right_wheel">
-    <visual>
-      <origin xyz="0 0 0"/>
-      <geometry>
-        <cylinder radius="0.05" length="0.04"/>
-      </geometry>
-      <material name="blue"/>
-    </visual>
-  </link>
-<!-- Définition du joint entre chassis et la roulette(caster_wheel) -->
-  <joint name="caster_wheel_joint" type="continuous">
-    <parent link="chassis"/>
-    <child link="caster_wheel"/>
-    <origin xyz="0.24 0 0" rpy="${pi/2} 0 0"/>
-  </joint>
-  <!-- Définition du lien la roulette(caster_wheel) -->
-  <link name="caster_wheel">
-    <visual>
-      <geometry>
-        <sphere radius="0.05" />
-      </geometry>
-      <material name="black"/>
-    </visual>
-  </link>
+<xacro:include filename="robot_core.xacro"/>
 </robot>
