Commit message: 

File: description/robot_core.xacro (robot description, xacro)
@@ -1,31 +1,40 @@
 <?xml version="1.0"?>
-<robot xmlns:xacro="http://www.ros.org/wiki/xacro"  >
-</material name="white">
-    <color rgba="1 1 1 1" />
-</material>
-</material name="orange">
-    <color rgba="1 0.3 0.1 1" />
-</material>
-</material name="blue">
-    <color rgba="0.2 0.2 1 1" />
-</material>
-</material name="black">
-    <color rgba="0 0 0 1" />
-</material>
-<link name="base_link">
-</link>
-<joint name="base_link" type="fixed">
+<robot xmlns:xacro="http://www.ros.org/wiki/xacro" name="robot">
+  <!-- Définition des matériaux -->
+  <material name="white">
+    <color rgba="1 1 1 1"/>
+  </material>
+  <material name="orange">
+    <color rgba="1 0.3 0.1 1"/>
+  </material>
+  <material name="blue">
+    <color rgba="0.2 0.2 1 1"/>
+  </material>
+  <material name="black">
+    <color rgba="0 0 0 1"/>
+  </material>
+  <!-- Définition du lien de base -->
+  <link name="base_link"/>
+  <!-- Définition du joint base_link -->
+  <joint name="base_joint" type="fixed">
+    <parent link="world"/>
+    <child link="base_link"/>
+    <origin xyz="0 0 0" rpy="0 0 0"/>
+  </joint>
+  <!-- Définition du lien chassis -->
+  <link name="chassis">
+    <visual>
+      <origin xyz="0.15 0 0.75"/>
+      <geometry>
+        <box size="0.3 0.3 0.15"/>
+      </geometry>
+      <material name="white"/>
+    </visual>
+  </link>
+  <!-- Définition du joint entre base_link et chassis -->
+  <joint name="chassis_joint" type="fixed">
     <parent link="base_link"/>
-    <child  link="chassis"/>
+    <child link="chassis"/>
     <origin xyz="-0.1 0 0"/>
-</joint>
-<link name="chassis">
-    <visual>
-        <origin xyz="0.15 0 0.75"/>
-        <geometry>
-            <box size="0.3 0.3 0.15"/>
-        </geometry>
-        <material name="white"/>
-    </visual>
-</link>
+  </joint>
 </robot>

Commit message: Ajout de modifications à file.txt

File: description/robot_core.xacro (robot description, xacro)
@@ -1,3 +1,4 @@
 <?xml version="1.0"?>
+<<<<<<< HEAD
 <robot xmlns:xacro="http://www.ros.org/wiki/xacro" name="robot">
   <!-- Définition des matériaux -->
@@ -39,2 +40,34 @@
   </joint>
 </robot>
+=======
+<robot xmlns:xacro="http://www.ros.org/wiki/xacro"  >
+</material name="white">
+    <color rgba="1 1 1 1" />
+</material>
+</material name="orange">
+    <color rgba="1 0.3 0.1 1" />
+</material>
+</material name="blue">
+    <color rgba="0.2 0.2 1 1" />
+</material>
+</material name="black">
+    <color rgba="0 0 0 1" />
+</material>
+<link name="base_link">
+</link>
+<joint name="base_link" type="fixed">
+    <parent link="base_link"/>
+    <child  link="chassis"/>
+    <origin xyz="-0.1 0 0"/>
+</joint>
+<link name="chassis">
+    <visual>
+        <origin xyz="0.15 0 0.75"/>
+        <geometry>
+            <box size="0.3 0.3 0.15"/>
+        </geometry>
+        <material name="white"/>
+    </visual>
+</link>
+</robot>
+>>>>>>> 20f9139 (Ajout de modifications à file.txt)

Commit message: Update robot_core.xacro and rsp.launch.py for articubot configuration

File: description/robot_core.xacro (robot description, xacro)
@@ -1,4 +1,3 @@
 <?xml version="1.0"?>
-<<<<<<< HEAD
 <robot xmlns:xacro="http://www.ros.org/wiki/xacro" name="robot">
   <!-- Définition des matériaux -->
@@ -16,5 +15,7 @@
   </material>
   <!-- Définition du lien de base -->
-  <link name="base_link"/>
+  <link name="base_link">
+    <!-- Contenu du lien base_link -->
+  </link>
   <!-- Définition du joint base_link -->
   <joint name="base_joint" type="fixed">
@@ -40,34 +41,2 @@
   </joint>
 </robot>
-=======
-<robot xmlns:xacro="http://www.ros.org/wiki/xacro"  >
-</material name="white">
-    <color rgba="1 1 1 1" />
-</material>
-</material name="orange">
-    <color rgba="1 0.3 0.1 1" />
-</material>
-</material name="blue">
-    <color rgba="0.2 0.2 1 1" />
-</material>
-</material name="black">
-    <color rgba="0 0 0 1" />
-</material>
-<link name="base_link">
-</link>
-<joint name="base_link" type="fixed">
-    <parent link="base_link"/>
-    <child  link="chassis"/>
-    <origin xyz="-0.1 0 0"/>
-</joint>
-<link name="chassis">
-    <visual>
-        <origin xyz="0.15 0 0.75"/>
-        <geometry>
-            <box size="0.3 0.3 0.15"/>
-        </geometry>
-        <material name="white"/>
-    </visual>
-</link>
-</robot>
->>>>>>> 20f9139 (Ajout de modifications à file.txt)

Commit message: couleur_chassis_gazebo

File: description/robot_core.xacro (robot description, xacro)
@@ -1,131 +1,125 @@
 <?xml version="1.0"?>
-<robot xmlns:xacro="http://www.ros.org/wiki/xacro" name="robot">
-  <xacro:include filename="inertial_macros.xacro"/>
-    <!-- Définition des matériaux -->
-  <material name="white">
-    <color rgba="1 1 1 1"/>
-  </material>
-  <material name="orange">
-    <color rgba="1 0.3 0.1 1"/>
-  </material>
-  <material name="blue">
-    <color rgba="0.2 0.2 1 1"/>
-  </material>
-  <material name="black">
-    <color rgba="0 0 0 1"/>
-  </material>
-  <!-- Définition du lien world -->
-  <link name="world">
-    <!-- Contenu du lien world -->
-  </link>
-  <!-- Définition du lien de base -->
-  <link name="base_link">
-    <!-- Contenu du lien base_link -->
-  </link>
-  <!-- Définition du joint base_joint -->
-  <joint name="base_joint" type="fixed">
-    <parent link="world"/>
-    <child link="base_link"/>
-    <origin rpy="0 0 0" xyz="0 0 0"/>
-  </joint>
-  <!-- Définition du lien chassis -->
-  <link name="chassis">
-    <visual>
-      <origin xyz="0.15 0 0.075"/>
-      <geometry>
-        <box size="0.3 0.3 0.15"/>
-      </geometry>
-      <material name="white"/>
-    </visual>
-    <collision>
-      <origin xyz="0.15 0 0.075"/>
-      <geometry>
-        <box size="0.3 0.3 0.15"/>
-      </geometry>
-    </collision>
-    <xacro:inertial_box mass="0.5" x="0.3" y="0.3" z="0.15">
-      <origin xyz="0.15 0 0.075" rpy="0 0 0"/>
-      </xacro:inertial_box>
-  </link>
-  <!-- Définition du joint entre base_link et chassis -->
-  <joint name="chassis_joint" type="fixed">
-    <parent link="base_link"/>
-    <child link="chassis"/>
-    <origin xyz="-0.1 0 0"/>
-  </joint>
-  <!-- Définition du joint entre chassis et le bras gauche -->
-  <joint name="left_wheel_joint" type="continuous">
-    <parent link="base_link"/>
-    <child link="left_wheel"/>
-    <origin xyz="0 0.175 0" rpy="-${pi/2} 0 0"/>
-    <axis xyz="0 0 1"/>
-  </joint>
-  <!-- Définition du lien bras gauche du chassis -->
-  <link name="left_wheel">
-    <visual>
-      <origin xyz="0 0 0"/>
-      <geometry>
-        <cylinder radius="0.05" length="0.04"/>
-      </geometry>
-      <material name="blue"/>
-    </visual>
-    <collision>
-      <origin xyz="0 0 0"/>
-      <geometry>
-        <cylinder radius="0.05" length="0.04"/>
-      </geometry>
-    </collision>
-    <xacro:inertial_cylinder mass="0.1" length="0.04" radius="0.05">
-      <origin xyz="0 0 0" rpy="0 0 0"/>
-    </xacro:inertial_cylinder>
-  </link>
-  <!-- Définition du joint entre chassis et le bras droit -->
-  <joint name="right_wheel_joint" type="continuous">
-    <parent link="base_link"/>
-    <child link="right_wheel"/>
-    <origin xyz="0 -0.175 0" rpy="${pi/2} 0 0"/>
-    <axis xyz="0 0 -1"/>
-  </joint>
-  <!-- Définition du lien bras droit du chassis -->
-  <link name="right_wheel">
-    <visual>
-      <origin xyz="0 0 0"/>
-      <geometry>
-        <cylinder radius="0.05" length="0.04"/>
-      </geometry>
-      <material name="blue"/>
-    </visual>
-    <collision>
-      <origin xyz="0 0 0"/>
-      <geometry>
-        <cylinder radius="0.05" length="0.04"/>
-      </geometry>
-    </collision>
-    <xacro:inertial_cylinder mass="0.1" length="0.04" radius="0.05">
-      <origin xyz="0 0 0" rpy="0 0 0"/>
-    </xacro:inertial_cylinder>
-  </link>
-<!-- Définition du joint entre chassis et la roulette(caster_wheel) -->
-  <joint name="caster_wheel_joint" type="continuous">
-    <parent link="chassis"/>
-    <child link="caster_wheel"/>
-    <origin xyz="0.24 0 0" rpy="${pi/2} 0 0"/>
-  </joint>
-  <!-- Définition du lien la roulette(caster_wheel) -->
-  <link name="caster_wheel">
-    <visual>
-      <geometry>
-        <sphere radius="0.05" />
-      </geometry>
-      <material name="black"/>
-    </visual>
-    <collision>
-      <geometry>
-        <sphere radius="0.05" />
-      </geometry>
-    </collision>
-    <xacro:inertial_sphere mass="0.1"  radius="0.05">
-      <origin xyz="0 0 0" rpy="0 0 0"/>
-    </xacro:inertial_sphere>
-  </link>
+<robot xmlns:xacro="http://www.ros.org/wiki/xacro" >
+    <xacro:include filename="inertial_macros.xacro"/>
+    <material name="white">
+        <color rgba="1 1 1 1" />
+    </material>
+    <material name="orange">
+        <color rgba="1 0.3 0.1 1"/>
+    </material>
+    <material name="blue">
+        <color rgba="0.2 0.2 1 1"/>
+    </material>
+    <material name="black">
+        <color rgba="0 0 0 1"/>
+    </material>
+    <!-- BASE LINK -->
+    <link name="base_link">
+    </link>
+    <!-- CHASSIS LINK -->
+    <joint name="chassis_joint" type="fixed">
+        <parent link="base_link"/>
+        <child link="chassis"/>
+        <origin xyz="-0.1 0 0"/>
+    </joint>
+    <link name="chassis">
+        <visual>
+            <origin xyz="0.15 0 0.075"/>
+            <geometry>
+                <box size="0.3 0.3 0.15"/>
+            </geometry>
+            <material name="white"/>
+        </visual>
+        <collision>
+            <origin xyz="0.15 0 0.075"/>
+            <geometry>
+                <box size="0.3 0.3 0.15"/>
+            </geometry>
+        </collision>
+        <xacro:inertial_box mass="0.5" x="0.3" y="0.3" z="0.15">
+            <origin xyz="0.15 0 0.075" rpy="0 0 0"/>
+        </xacro:inertial_box>
+    </link>
+    <gazebo reference="chassis">
+        <material>Gazebo/White</material>
+    </gazebo>
+    <!-- LEFT WHEEL LINK -->
+    <joint name="left_wheel_joint" type="continuous">
+        <parent link="base_link"/>
+        <child link="left_wheel"/>
+        <origin xyz="0 0.175 0" rpy="-${pi/2} 0 0" />
+        <axis xyz="0 0 1"/>
+    </joint>
+    <link name="left_wheel">
+        <visual>
+            <geometry>
+                <cylinder radius="0.05" length="0.04"/>
+            </geometry>
+            <material name="blue"/>
+        </visual>
+        <collision>
+            <geometry>
+                <cylinder radius="0.05" length="0.04"/>
+            </geometry>
+        </collision>
+        <xacro:inertial_cylinder mass="0.1" length="0.04" radius="0.05">
+            <origin xyz="0 0 0" rpy="0 0 0"/>
+        </xacro:inertial_cylinder>
+    </link>
+    <gazebo reference="left_wheel">
+        <material>Gazebo/Blue</material>
+    </gazebo>
+    <!-- RIGHT WHEEL LINK -->
+    <joint name="right_wheel_joint" type="continuous">
+        <parent link="base_link"/>
+        <child link="right_wheel"/>
+        <origin xyz="0 -0.175 0" rpy="${pi/2} 0 0" />
+        <axis xyz="0 0 -1"/>
+    </joint>
+    <link name="right_wheel">
+        <visual>
+            <geometry>
+                <cylinder radius="0.05" length="0.04"/>
+            </geometry>
+            <material name="blue"/>
+        </visual>
+        <collision>
+            <geometry>
+                <cylinder radius="0.05" length="0.04"/>
+            </geometry>
+        </collision>
+        <xacro:inertial_cylinder mass="0.1" length="0.04" radius="0.05">
+            <origin xyz="0 0 0" rpy="0 0 0"/>
+        </xacro:inertial_cylinder>
+    </link>
+    <gazebo reference="right_wheel">
+        <material>Gazebo/Blue</material>
+    </gazebo>
+    <!-- CASTER WHEEL LINK -->
+    <joint name="caster_wheel_joint" type="fixed">
+        <parent link="chassis"/>
+        <child link="caster_wheel"/>
+        <origin xyz="0.24 0 0"/>
+    </joint>
+    <link name="caster_wheel">
+        <visual>
+            <geometry>
+                <sphere radius="0.05"/>
+            </geometry>
+            <material name="black"/>
+        </visual>
+        <collision>
+            <geometry>
+                <sphere radius="0.05"/>
+            </geometry>
+        </collision>
+        <xacro:inertial_sphere mass="0.1" radius="0.05">
+            <origin xyz="0 0 0" rpy="0 0 0"/>
+        </xacro:inertial_sphere>
+    </link>
+    <gazebo reference="caster_wheel">
+        <material>Gazebo/Black</material>
+        <mu1 value="0.001"/>
+        <mu2 value="0.001"/>
+    </gazebo>
 </robot>
